Commit message: Remove the "_link" suffix from link names in the URDF UR5 model

File: tests/models/ur5/ur5-gmv.urdf (robot description, URDF)
Before this commit: robot ur5, 13 links, 12 joints
Links:
- removed link base_link
- removed link forearm_link
- removed link shoulder_link
- removed link upper_arm_link
- removed link wrist_1_link
- removed link wrist_2_link
- removed link wrist_3_link
- added link base_dummy
- added link forearm, mass 2.275
- added link shoulder, mass 3.7
- added link upper_arm, mass 8.393
- added link wrist_1, mass 1.219
- added link wrist_2, mass 1.219
- added link wrist_3, mass 0.1879
- link base: mass None -> 4.0
Joints:
- joint base_link-base_fixed_joint: child base -> base_dummy; parent base_link -> base
- joint elbow_joint: child forearm_link -> forearm; parent upper_arm_link -> upper_arm
- joint plate_fixed_joint: parent wrist_3_link -> wrist_3
- joint shoulder_lift_joint: child upper_arm_link -> upper_arm; parent shoulder_link -> shoulder
- joint shoulder_pan_joint: child shoulder_link -> shoulder; parent base_link -> base
- joint world_joint: child base_link -> base
- joint wrist_1_joint: child wrist_1_link -> wrist_1; parent forearm_link -> forearm
- joint wrist_2_joint: child wrist_2_link -> wrist_2; parent wrist_1_link -> wrist_1
- joint wrist_3_joint: child wrist_3_link -> wrist_3; parent wrist_2_link -> wrist_2
- joint wrist_3_link-tool0_fixed_joint: parent wrist_3_link -> wrist_3
